Commit message: Add ros_control into example simulation

File: example/robots/simple_robot.xacro (robot description, xacro)
@@ -68,5 +68,5 @@
     <child link="top"/>
     <axis xyz="0.0 0.0 1.0"/>
-    <limit effort="10.0" lower="-1000000000.0" upper="1000000000.0" velocity="100.0"/>
+    <limit effort="100.0" lower="-100000.0" upper="100000.0" velocity="10.0"/>
   </joint>
   <joint name="joint_pointer" type="fixed">
@@ -76,4 +76,14 @@
     <axis xyz="0.0 0.0 0.0"/>
   </joint>
+  <transmission name="simple_transmission">
+    <type>transmission_interface/SimpleTransmission</type>
+    <joint name="joint">
+      <hardwareInterface>hardware_interface/PositionJointInterface</hardwareInterface>
+    </joint>
+    <actuator name="motor">
+      <hardwareInterface>hardware_interface/PositionJointInterface</hardwareInterface>
+      <mechanicalReduction>1</mechanicalReduction>
+    </actuator>
+  </transmission>
   <gazebo reference="top">
     <material>Gazebo/Red</material>
@@ -85,3 +95,8 @@
     <material>Gazebo/Yellow</material>
   </gazebo>
+  <gazebo>
+    <plugin name="gazebo_ros_control" filename="libgazebo_ros_control.so">
+      <robotNamespace>/simple_robot</robotNamespace>
+    </plugin>
+  </gazebo>
 </robot>
